File: USB Sensor/Display_LED.sch (EAGLE design)
At the start: 7 parts, among them U1 ATMEGA644M, U3 TLV61220DBV

Commit message: Continued layout of display module
Preliminary placement done, major layout remaining
Parts:
- removed L2: 6.8uH, bschulz:INDUCTOR1008
- removed U3: TLV61220DBV, bschulz:TLV61220DBV
- added BT1: AACLIP, bschulz:AACLIP
- added C10, C13, C5: 1uF, bschulz_passives:C-EU1UFC0603
- added C11: 0.1uF, bschulz_passives:C-EU1UFC0603
- added C12, C3, C4: 0.1uF, bschulz_passives:C-EU0.1UFC0603
- added C6: 10uF, bschulz_passives:C-EU10UFC0805
- added C7: 10pF, bschulz_passives:C-EU10PFC0603
- added C8, C9: 4.7uF, bschulz_passives:C-EU4.7UFC0805
- added D1, D10, D11, D12, D13, D2, D3, D4, D5, D6, D7, D8, D9: LED0603, bschulz:LED0603
- added ISP1, ISP2, ISP4: AVRISP-6, bschulz:AVRISP-6
- added J1: (no value), bschulz:CONN_2X2MIRCOFIT_RT
- added L1: (no value), bschulz:INDUCTORMAPI_3X3
- added LED1, LED4: YSD-439AR6B-35, SparkFun-LED:7-SEGMENT-4DIGIT-10MM-RED
- added Q1, Q13, Q14, Q15, Q16, Q2, Q3, Q4: MOSFET-NCH-2N7002P, bschulz:MOSFET-NCH-2N7002P
- added Q5: MOSFET-NCH-ZXMN3B14FTA, bschulz:MOSFET-NCH-ZXMN3B14FTA
- added R10, R22, R24, R3, R4, R5, R6, R7, R8, R9: 100k, bschulz_passives:R-EU_100KR0603
- added R11, R37, R45: 10k, bschulz_passives:R-EU_10KR0603
- added R12, R13, R14, R15, R16, R17, R18, R19, R20, R21, R26, R27, R28, R29, R30, R31, R32, R33, R35, R36, R38, R39, R46, R47, R48, R49, R50, R51, R52, R53, R54, R55: (no value), bschulz_passives:R-EU_330R0603
- added R23: 316k, bschulz_passives:R-EU_316KR0603
- added R25: (no value), bschulz_passives:R-EU_10KR0603
- added R34: 330R, bschulz_passives:R-EU_330R0603
- added S1: DIP_8219_GULL, bschulz:DIP_8219_GULL
- added S2, S3, S4: BUTTON6X6, bschulz:BUTTON6X6
- added S5: SPDTOS1020, bschulz:SPDTOS1020
- added U2: (no value), bschulz:SN74HC165PW
- added U4, U7: ATMEGA48PMLF, bschulz:ATMEGA48PMLF
- added U5: TPS61021A, bschulz:TPS61021A
- added XTAL1: CRYSTAL8MHZ5X3.2, bschulz:CRYSTAL8MHZ5X3.2
- C1, C2: value 10uF -> (none); device bschulz_passives:C-EU10UFC0805 -> bschulz_passives:C-EU12PFC0402
- R1: value 1M -> (none); device bschulz_passives:R-EU_1MR0603 -> bschulz_passives:R-EU_10KR0603
- R2: value 180k -> (none); device bschulz_passives:R-EU_180KR0603 -> bschulz_passives:R-EU_10KR0603
Connections:
- removed net FB1: R1.1, R2.2, U3.FB
- removed net RX0: U1.(PCINT24/RXD0)PD0
- removed net SW1: L2.2, U3.SW
- removed net TX0: U1.(PCINT25/TXD0)PD1
- removed net VIN: C1.1, L2.1, U3.EN, U3.VBAT
- new net !RESET: ISP2.RST, R37.1, U1.RESET
- new net !RESET_A: ISP1.RST, R11.1, U4.(PCINT14/!RESET!)PC6
- new net !RESET_B: ISP4.RST, R45.1, U7.(PCINT14/!RESET!)PC6
- new net B0: R3.1, S1.16, U2.A
- new net B1: R4.1, S1.15, U2.B
- new net B2: R5.1, S1.14, U2.C
- new net B3: R6.1, S1.13, U2.D
- new net B4: R7.1, S1.12, U2.E
- new net B5: R8.1, S1.11, U2.F
- new net B6: R9.1, S1.10, U2.G
- new net B7: R10.1, S1.9, U2.H
- new net BAT: BT1.+, C6.1, L1.1, Q5.G, R34.2, S5.O, U5.VIN
- new net BOOST_EN: R22.2, S5.P, U5.EN
- new net DIP_CLK: U1.(PCINT5/ADC5)PA5, U2.CLK
- new net DIP_LD: U1.(PCINT6/ADC6)PA6, U2.SH/!LD
- new net DIP_OUT: U1.(PCINT4/ADC4)PA4, U2.QH
- new net DISP_SEL_A: R1.1, S2.1, S2.2, U1.(PCINT22/TOSC1)PC6
- new net DISP_SEL_B: R2.1, S3.1, S3.2, U1.(PCINT23/TOSC2)PC7
- new net DISP_STAT_D1_A: R28.2, U1.(PCINT29/OC1A)PD5
- new net DISP_STAT_D1_B: R32.2, U1.(PCINT19/TMS)PC3
- new net DISP_STAT_D2_A: R29.2, U1.(PCINT28/OC1B)PD4
- new net DISP_STAT_D2_B: R33.2, U1.(PCINT18/TCK)PC2
- new net DISP_STAT_I_A: R27.2, U1.(PCINT30/OC2B/ICP)PD6
- new net DISP_STAT_I_B: R31.2, U1.(PCINT20/TDO)PC4
- new net DISP_STAT_V_A: R26.2, U1.(PCINT31/OC2A)PD7
- new net DISP_STAT_V_B: R30.2, U1.(PCINT21/TDI)PC5
- new net DIS_A1: LED1.A, R12.1
- new net DIS_A2: LED4.A, R46.1
- new net DIS_B1: LED1.B, R13.1
- new net DIS_B2: LED4.B, R47.1
- new net DIS_C1: LED1.C, R14.1
- new net DIS_C2: LED4.C, R48.1
- new net DIS_COL1: LED1.COL-C, R20.1
- new net DIS_COL2: LED4.COL-C, R54.1
- new net DIS_D1: LED1.D, R15.1
- new net DIS_D2: LED4.D, R49.1
- new net DIS_DIG1_1: LED1.DIG1, Q1.D
- new net DIS_DIG1_2: LED4.DIG1, Q13.D
- new net DIS_DIG2_1: LED1.DIG2, Q2.D
- new net DIS_DIG2_2: LED4.DIG2, Q14.D
- new net DIS_DIG3_1: LED1.DIG3, Q3.D
- new net DIS_DIG3_2: LED4.DIG3, Q15.D
- new net DIS_DIG4_1: LED1.DIG4, Q4.D
- new net DIS_DIG4_2: LED4.DIG4, Q16.D
- new net DIS_DP1: LED1.DP, R19.1
- new net DIS_DP2: LED4.DP, R53.1
- new net DIS_E1: LED1.E, R16.1
- new net DIS_E2: LED4.E, R50.1
- new net DIS_F1: LED1.F, R17.1
- new net DIS_F2: LED4.F, R51.1
- new net DIS_G1: LED1.G, R18.1
- new net DIS_G2: LED4.G, R52.1
- new net DIS_POS1: LED1.APOS-C, R21.1
- new net DIS_POS2: LED4.APOS-C, R55.1
- new net FB: C7.2, R23.1, R24.2, U5.FB
- new net HOLD: R25.1, S4.1, S4.2, U1.(PCINT7/ADC7)PA7
- new net MCU_A1: R12.2, U4.(PCINT18/INT0)PD2
- new net MCU_A2: R46.2, U7.(PCINT18/INT0)PD2
- new net MCU_B1: R13.2, U4.(PCINT19/INT1)PD3
- new net MCU_B2: R47.2, U7.(PCINT19/INT1)PD3
- new net MCU_C1: R14.2, U4.(PCINT20/XCK/T0)PD4
- new net MCU_C2: R48.2, U7.(PCINT20/XCK/T0)PD4
- new net MCU_COL1: R20.2, U4.(PCINT0/CLKO/ICP1)PB0
- new net MCU_COL2: R54.2, U7.(PCINT0/CLKO/ICP1)PB0
- new net MCU_D1: R15.2, U4.(PCINT21/OC0B/T1)PD5
- new net MCU_D2: R49.2, U7.(PCINT21/OC0B/T1)PD5
- new net MCU_DIG1_1: Q1.G, U4.(PCINT11/ADC3)PC3
- new net MCU_DIG1_2: Q13.G, U7.(PCINT11/ADC3)PC3
- new net MCU_DIG2_1: Q2.G, U4.(PCINT10/ADC2)PC2
- new net MCU_DIG2_2: Q14.G, U7.(PCINT10/ADC2)PC2
- new net MCU_DIG3_1: Q3.G, U4.(PCINT9/ADC1)PC1
- new net MCU_DIG3_2: Q15.G, U7.(PCINT9/ADC1)PC1
- new net MCU_DIG4_1: Q4.G, U4.(PCINT8/ADC0)PC0
- new net MCU_DIG4_2: Q16.G, U7.(PCINT8/ADC0)PC0
- new net MCU_DP1: R19.2, U4.(PCINT2/!SS!/OC1B)PB2
- new net MCU_DP2: R53.2, U7.(PCINT2/!SS!/OC1B)PB2
- new net MCU_E1: R16.2, U4.(PCINT22/OC0A/AIN0)PD6
- new net MCU_E2: R50.2, U7.(PCINT22/OC0A/AIN0)PD6
- new net MCU_F1: R17.2, U4.(PCINT23/AIN1)PD7
- new net MCU_F2: R51.2, U7.(PCINT23/AIN1)PD7
- new net MCU_G1: R18.2, U4.(PCINT6/XTAL1/TOSC1)PB6
- new net MCU_G2: R52.2, U7.(PCINT6/XTAL1/TOSC1)PB6
- new net MCU_POS1: R21.2, U4.(PCINT1/OC1A)PB1
- new net MCU_POS2: R55.2, U7.(PCINT1/OC1A)PB1
- new net MISO_A: ISP1.MISO, U4.(PCINT4/MISO)PB4
- new net MISO_B: ISP4.MISO, U7.(PCINT4/MISO)PB4
- new net MOSI_A: ISP1.MOSI, U4.(PCINT3/OC2A/MOSI)PB3
- new net MOSI_B: ISP4.MOSI, U7.(PCINT3/OC2A/MOSI)PB3
- new net N$1: D1.ANODE, R26.1
- new net N$10: BT1.-, D9.ANODE, Q5.D
- new net N$11: D9.CATHODE, R34.1
- new net N$12: D12.ANODE, R38.1
- new net N$13: C2.2, U1.XTAL1, XTAL1.1
- new net N$14: D11.ANODE, R36.1
- new net N$15: C1.2, U1.XTAL2, XTAL1.2
- new net N$16: D13.ANODE, R39.1
- new net N$2: D2.ANODE, R27.1
- new net N$21: U1.(PCINT3/ADC3)PA3
- new net N$22: U1.(PCINT2/ADC2)PA2
- new net N$23: U1.(PCINT1/ADC1)PA1
- new net N$24: U1.(PCINT0/ADC0)PA0
- new net N$3: D3.ANODE, R28.1
- new net N$4: D4.ANODE, R29.1
- new net N$5: D5.ANODE, R30.1
- new net N$6: D6.ANODE, R31.1
- new net N$7: D7.ANODE, R32.1
- new net N$8: D8.ANODE, R33.1
- new net N$9: D10.ANODE, R35.1
- new net PG: R36.2
- new net RX2: U1.(PCINT27/INT1)PD3, U7.(PCINT16/RXD)PD0
- new net SCK_A: ISP1.SCK, U4.(PCINT5/SCK)PB5
- new net SCK_B: ISP4.SCK, U7.(PCINT5/SCK)PB5
- new net STAT1: R39.2
- new net STAT2: R38.2
- new net SW: L1.2, U5.SW
- new net TX2: U1.(PCINT26/INT0)PD2, U7.(PCINT17/TXD)PD1
- net 3V3: now also C10.1, C11.1, C12.1, C13.1, C3.1, C4.1, C5.1, C7.1, C8.1, C9.1, ISP1.VCC, ISP2.VCC, ISP4.VCC, R10.2, R11.2, R2.2, R23.2, R25.2, R3.2, R35.2, R37.2, R4.2, R45.2, R5.2, R6.2, R7.2, R8.2, R9.2, U1.AREF, U1.AVCC, U1.VCC, U1.VCC@1, U1.VCC@2, U2.VCC, U4.AREF, U4.AVCC, U4.VCC, U5.VOUT, U7.AREF, U7.AVCC, U7.VCC; no longer C2.1, U3.VOUT
- net GND: now also C1.1, C10.2, C11.2, C12.2, C13.2, C2.1, C3.2, C4.2, C5.2, C6.2, C8.2, C9.2, D1.CATHODE, D10.CATHODE, D11.CATHODE, D12.CATHODE, D13.CATHODE, D2.CATHODE, D3.CATHODE, D4.CATHODE, D5.CATHODE, D6.CATHODE, D7.CATHODE, D8.CATHODE, ISP1.GND, ISP2.GND, ISP4.GND, LED1.APOS-A, LED1.COL-A, LED4.APOS-A, LED4.COL-A, Q1.S, Q13.S, Q14.S, Q15.S, Q16.S, Q2.S, Q3.S, Q4.S, Q5.S, R22.1, R24.1, S1.1, S1.2, S1.3, S1.4, S1.5, S1.6, S1.7, S1.8, S2.3, S2.4, S3.3, S3.4, S4.3, S4.4, S5.S, U1.EXP, U1.GND, U1.GND@1, U1.GND@2, U1.GND@3, U2.GND, U2.SER, U4.GND, U5.AGND, U5.PGND, U7.GND; no longer C1.2, C2.2, R2.1, U3.GND
- net MISO: now also ISP2.MISO
- net MOSI: now also ISP2.MOSI
- net RX1: now also U1.(PCINT25/TXD0)PD1, U4.(PCINT16/RXD)PD0; no longer U1.(PCINT26/INT0)PD2
- net SCK: now also ISP2.SCK
- net TX1: now also U1.(PCINT24/RXD0)PD0, U4.(PCINT17/TXD)PD1; no longer U1.(PCINT27/INT1)PD3
Other:
- note added: "Allow for additional bulk capacitance if needed"
- note added: "BAT - Analog PG - DO DIP_LD - DO DIP_CLK - DO DIP_OUT - DI DISP_SEL_A - DI DISP_SEL_B - DI HOLD - DI STAT1 - DO STAT2- DO"
- moved on the sheet: C1, C2, R1, R2

Commit message: Display layout complete, review required
Layout of display module is complete, should be reviewed before sending to fab
Parts:
- removed LED1, LED4: YSD-439AR6B-35, SparkFun-LED:7-SEGMENT-4DIGIT-10MM-RED
- added DS1, DS2: YSD-439AK2B-35, bschulz:LED_7-SEGMENT-4DIGIT-10MM-KGREEN
- added H1, H2, H3, H4, H5: (no value), bschulz:MOUNTING_HOLE2_NP
- added R40: (no value), bschulz_passives:R-EU_1KR0603
- renumbered ISP4 to ISP3
Connections:
- removed net N$21: U1.(PCINT3/ADC3)PA3
- removed net N$22: U1.(PCINT2/ADC2)PA2
- removed net N$23: U1.(PCINT1/ADC1)PA1
- removed net N$24: U1.(PCINT0/ADC0)PA0
- new net BAT_SENSE: R40.1, U1.(PCINT0/ADC0)PA0
- net !RESET: now also ISP1.RST; no longer ISP2.RST
- net !RESET_A: now also ISP2.RST; no longer ISP1.RST
- net 3V3: now also J1.1
- net BAT: now also R40.2
- net DIS_A1: now also DS1.A; no longer LED1.A
- net DIS_A2: now also DS2.A; no longer LED4.A
- net DIS_B1: now also DS1.B; no longer LED1.B
- net DIS_B2: now also DS2.B; no longer LED4.B
- net DIS_C1: now also DS1.C; no longer LED1.C
- net DIS_C2: now also DS2.C; no longer LED4.C
- net DIS_COL1: now also DS1.COL-C; no longer LED1.COL-C
- net DIS_COL2: now also DS2.COL-C; no longer LED4.COL-C
- net DIS_D1: now also DS1.D; no longer LED1.D
- net DIS_D2: now also DS2.D; no longer LED4.D
- net DIS_DIG1_1: now also DS1.DIG1; no longer LED1.DIG1
- net DIS_DIG1_2: now also DS2.DIG1; no longer LED4.DIG1
- net DIS_DIG2_1: now also DS1.DIG2; no longer LED1.DIG2
- net DIS_DIG2_2: now also DS2.DIG2; no longer LED4.DIG2
- net DIS_DIG3_1: now also DS1.DIG3; no longer LED1.DIG3
- net DIS_DIG3_2: now also DS2.DIG3; no longer LED4.DIG3
- net DIS_DIG4_1: now also DS1.DIG4; no longer LED1.DIG4
- net DIS_DIG4_2: now also DS2.DIG4; no longer LED4.DIG4
- net DIS_DP1: now also DS1.DP; no longer LED1.DP
- net DIS_DP2: now also DS2.DP; no longer LED4.DP
- net DIS_E1: now also DS1.E; no longer LED1.E
- net DIS_E2: now also DS2.E; no longer LED4.E
- net DIS_F1: now also DS1.F; no longer LED1.F
- net DIS_F2: now also DS2.F; no longer LED4.F
- net DIS_G1: now also DS1.G; no longer LED1.G
- net DIS_G2: now also DS2.G; no longer LED4.G
- net DIS_POS1: now also DS1.APOS-C; no longer LED1.APOS-C
- net DIS_POS2: now also DS2.APOS-C; no longer LED4.APOS-C
- net GND: now also DS1.APOS-A, DS1.COL-A, DS2.APOS-A, DS2.COL-A, J1.2; no longer LED1.APOS-A, LED1.COL-A, LED4.APOS-A, LED4.COL-A
- net MISO: now also ISP1.MISO; no longer ISP2.MISO
- net MISO_A: now also ISP2.MISO; no longer ISP1.MISO
- net MOSI: now also ISP1.MOSI; no longer ISP2.MOSI
- net MOSI_A: now also ISP2.MOSI; no longer ISP1.MOSI
- net PG: now also U1.(PCINT1/ADC1)PA1
- net SCK: now also ISP1.SCK; no longer ISP2.SCK
- net SCK_A: now also ISP2.SCK; no longer ISP1.SCK
- net SCL: now also J1.3
- net SDA: now also J1.4
- net STAT1: now also U1.(PCINT2/ADC2)PA2
- net STAT2: now also U1.(PCINT3/ADC3)PA3
Other:
- moved on the sheet: ISP1, ISP2
