File: USB Sensor/USBA1P_0v0.brd (EAGLE design)
At the start: 33 x 17.4 mm, 13 parts, among them J1 USBA_FEMALE_AMPHENOL, J2 USBA_MALE_MOLEX, U1 PAC1710

Commit message: Minor cleanup for USBA1P and USBm1P
Cleanup to part naming and layout for A1P and micro setups
Parts:
- J1: device bschulz:USB_A_AMPHENOL -> bschulz:USB_A_FEMALE_AMPHENOL
- J2: device bschulz:USB_A_0480372200 -> bschulz:USB_A_MALE_0480372200
Changed lines of the file:
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@@
 <layer number="27" name="tValues" color="7" fill="1" visible="no" active="yes"/>
 <layer number="28" name="bValues" color="7" fill="1" visible="no" active="yes"/>
-<layer number="29" name="tStop" color="7" fill="3" visible="no" active="yes"/>
+<layer number="29" name="tStop" color="7" fill="3" visible="yes" active="yes"/>
 <layer number="30" name="bStop" color="7" fill="6" visible="no" active="yes"/>
 <layer number="31" name="tCream" color="7" fill="4" visible="no" active="yes"/>
@@
 </autorouter>
 <elements>
-<element name="J1" library="bschulz" package="USB_A_AMPHENOL" value="USBA_FEMALE_AMPHENOL" x="22.86" y="8.636" smashed="yes" rot="R270">
+<element name="J1" library="bschulz" package="USB_A_FEMALE_AMPHENOL" value="USBA_FEMALE_AMPHENOL" x="22.86" y="8.636" smashed="yes" rot="R270">
 <attribute name="DIGIKEY" value="UE27AC54100-ND" x="-1.27" y="-12.954" size="1.778" layer="27" rot="R270" display="off"/>
 <attribute name="MF" value="Amphenol" x="-1.27" y="-12.954" size="1.778" layer="27" rot="R270" display="off"/>
@@
 <attribute name="NAME" x="30.226" y="16.637" size="0.8128" layer="25" font="vector" ratio="15" align="center"/>
 </element>
-<element name="J2" library="bschulz" package="USB_A_0480372200" value="USBA_MALE_MOLEX" x="4.064" y="8.636" smashed="yes" rot="R270">
+<element name="J2" library="bschulz" package="USB_A_MALE_0480372200" value="USBA_MALE_MOLEX" x="4.064" y="8.636" smashed="yes" rot="R270">
 <attribute name="DIGIKEY" value="WM3983CT-ND" x="-14.986" y="-11.684" size="1.778" layer="27" rot="R270" display="off"/>
 <attribute name="MF" value="Molex" x="-14.986" y="-11.684" size="1.778" layer="27" rot="R270" display="off"/>
